Commit message: renamed joints

File: joints/R105/description/urdf/R105.urdf.xacro (robot description, xacro)
@@ -2,13 +2,13 @@
 <robot xmlns:xacro="http://www.ros.org/wiki/xacro">
   <!-- <xacro:property name="joint_material" value="0.019608 0.32549 1 1" /> -->
-  <xacro:macro name="revolute_m" params="prefix parent_connection input *origin
+    <xacro:macro name="R105" params="prefix parent_connection input *origin
       mass='1.6'
       ixx='0.005898' ixy='0' ixz='0' iyy='0.003584' iyz='0.000096' izz='0.005765'
       effort='10' velocity='1' lower='-3.141593' upper='3.141593'">
       <!-- Actual joint geometry -->
-      <link name="${prefix}_revolute_m_link">
+      <link name="${prefix}_R105_link">
         <visual>
           <origin xyz="0 0 0" rpy="1.570796 0 0" />
-          <geometry><mesh filename="file://$(find revolute_m_description)/meshes/revolute_m_visual.glb" /></geometry>
+          <geometry><mesh filename="file://$(find R105_description)/meshes/R105_visual.glb" /></geometry>
           <!-- <material name="joint_material" /> -->
         </visual>
@@ -26,5 +26,5 @@
       <joint name="${prefix}" type="revolute">
         <origin xyz="0 0.09873 0" rpy="1.570796 1.570796 0.0" />
-        <parent link="${prefix}_revolute_m_link" />
+        <parent link="${prefix}_R105_link" />
         <child link="${prefix}_joint_out" />
         <axis xyz="0 0 1" />
@@ -34,5 +34,5 @@
         <origin xyz="0 0 0.06257" rpy="0 0 -1.570796" />
         <parent link="${prefix}_joint_in" />
-        <child link="${prefix}_revolute_m_link" />
+        <child link="${prefix}_R105_link" />
       </joint>
       <!-- Empty links to attach child joints to the input or output of this joint -->

File: joints/R120/description/urdf/R120.urdf.xacro (robot description, xacro)
@@ -2,17 +2,17 @@
 <robot xmlns:xacro="http://www.ros.org/wiki/xacro">
   <!-- <xacro:property name="joint_material" value="0.019608 0.32549 1 1" /> -->
-  <xacro:macro name="revolute_l" params="prefix parent_connection input *origin
+  <xacro:macro name="R120" params="prefix parent_connection input *origin
       mass='1.6'
       ixx='0.005898' ixy='0' ixz='0' iyy='0.003584' iyz='0.000096' izz='0.005765'
       effort='10' velocity='1' lower='-3.141593' upper='3.141593'">
       <!-- Actual joint geometry -->
-      <link name="${prefix}_revolute_l_link">
+      <link name="${prefix}_R120_link">
         <visual>
           <origin xyz="0 0 0" rpy="1.570796 0 0" />
-          <geometry><mesh filename="file://$(find revolute_l_description)/meshes/revolute_l_visual.glb" /></geometry>
+          <geometry><mesh filename="file://$(find R120_description)/meshes/R120_visual.glb" /></geometry>
           <!-- <material name="joint_material" /> -->
         </visual>
         <collision>
-          <geometry><mesh filename="file://$(find revolute_l_description)/meshes/revolute_l_collision.stl" /></geometry>
+          <geometry><mesh filename="file://$(find R120_description)/meshes/R120_collision.stl" /></geometry>
         </collision>
         <inertial>
@@ -23,5 +23,5 @@
       <joint name="${prefix}" type="revolute">
         <origin xyz="0 -0.088002 0" rpy="1.570796 1.570796 0.0" />
-        <parent link="${prefix}_revolute_l_link" />
+        <parent link="${prefix}_R120_link" />
         <child link="${prefix}_joint_out" />
         <axis xyz="0 0 1" />
@@ -31,5 +31,5 @@
         <origin xyz="0 0 0.070002" rpy="0 0 -1.570796" />
         <parent link="${prefix}_joint_in" />
-        <child link="${prefix}_revolute_l_link" />
+        <child link="${prefix}_R120_link" />
       </joint>
       <!-- Empty links to attach child joints to the input or output of this joint -->
