Commit message: .

File: joints/revolute_m/description/urdf/revolute_m.urdf.xacro (robot description, xacro)
@@ -25,5 +25,5 @@
       </link>
       <joint name="${prefix}" type="revolute">
-        <origin xyz="0 0.09873 0" rpy="1.570796 1.570796 0.0" />
+        <origin xyz="0 -0.09873 0" rpy="1.570796 1.570796 0.0" />
         <parent link="${prefix}_revolute_m_link" />
         <child link="${prefix}_joint_out" />
